Commit message: Fixed renaming

File: kaia_gazebo/urdf/kaia_snoopy.urdf (robot description, URDF)
Before this commit: robot kaia_burger, 7 links, 6 joints
Links:
- link base_link: geometry collision box size=0.140 0.140 0.143; visual mesh filename=package://kaia_gazebo/models/kaia_common/meshes/snoopy_base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 scale=0.001 0.001 0.001
